File: hardware/lemon-pepper.kicad_sch (KiCad schematic)
At the start: 21 parts, among them J101 INPUT, M101 MOT

Commit message: Update BOM field LCSC ID
Parts:
- C101, C102, C103, C104, C105, C106, C107, C108: LCSC ID (none) -> C440198; LCSC Part C440198 -> (none)
- D101: LCSC ID (none) -> C14996; LCSC Part C14996 -> (none)
- R101, R102: LCSC ID (none) -> C25905; LCSC Part C25905 -> (none)
- R103: LCSC ID (none) -> C25079; LCSC Part C25079 -> (none)
- R104, R105: LCSC ID (none) -> C17168; LCSC Part C17168 -> (none)
Changed lines of the file:
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@@
 			)
 		)
-		(property "LCSC Part" "C440198"
+		(property "LCSC ID" "C440198"
 			(at 127 182.88 0)
 			(effects
@@
 			)
 		)
-		(property "LCSC Part" "C440198"
+		(property "LCSC ID" "C440198"
 			(at 121.92 173.99 0)
 			(effects
@@
 			)
 		)
-		(property "LCSC Part" "C17168"
+		(property "LCSC ID" "C17168"
 			(at 82.55 92.71 0)
 			(effects
@@
 			)
 		)
-		(property "LCSC Part" "C17168"
+		(property "LCSC ID" "C17168"
 			(at 82.55 95.25 0)
 			(effects
@@
 			)
 		)
-		(property "LCSC Part" ""
-			(at 36.83 90.17 0)
-			(effects
-				(font
-					(size 1.27 1.27)
-				)
-				(hide yes)
-			)
-		)
 		(pin "1"
 		)
@@
 			)
 		)
-		(property "LCSC Part" "C440198"
+		(property "LCSC ID" "C440198"
 			(at 137.16 182.88 0)
 			(effects
@@
 			)
 		)
-		(property "LCSC Part" "C440198"
+		(property "LCSC ID" "C440198"
 			(at 142.24 173.99 0)
 			(effects
@@
 			)
 		)
-		(property "LCSC Part" ""
-			(at 269.24 130.81 0)
-			(effects
-				(font
-					(size 1.27 1.27)
-				)
-				(hide yes)
-			)
-		)
 		(pin "1"
 		)
@@
 			)
 		)
-		(property "LCSC Part" "C25079"
+		(property "LCSC ID" "C25079"
 			(at 58.42 110.49 0)
 			(effects
@@
 			)
 		)
-		(property "LCSC Part" "C14996"
+		(property "LCSC ID" "C14996"
 			(at 100.33 177.8 0)
 			(effects
@@
 			)
 		)
-		(property "LCSC Part" "C440198"
+		(property "LCSC ID" "C440198"
 			(at 106.68 182.88 0)
 			(effects
@@
 			)
 		)
-		(property "LCSC Part" "C440198"
+		(property "LCSC ID" "C440198"
 			(at 116.84 182.88 0)
 			(effects
@@
 			)
 		)
-		(property "LCSC Part" "C440198"
+		(property "LCSC ID" "C440198"
 			(at 132.08 173.99 0)
 			(effects
@@
 			)
 		)
-		(property "LCSC Part" "C25905"
+		(property "LCSC ID" "C25905"
 			(at 69.85 57.15 0)
 			(effects
@@
 			)
 		)
-		(property "LCSC Part" "C440198"
+		(property "LCSC ID" "C440198"
 			(at 111.76 173.99 0)
 			(effects
@@
 			)
 		)
-		(property "LCSC Part" "C25905"
+		(property "LCSC ID" "C25905"
 			(at 69.85 59.69 0)
 			(effects

Commit message: update to kicad 9
Changed lines of the file:
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@@
 (kicad_sch
-	(version 20231120)
+	(version 20250114)
 	(generator "eeschema")
-	(generator_version "8.0")
+	(generator_version "9.0")
 	(paper "A4")
 	(title_block
@@
 		(company "matei repair lab")
 	)
+	(text "this pinout should work\nfor all pre-wired steppers\nAABB\nABAB"
+		(exclude_from_sim no)
+		(at 255.27 121.92 0)
+		(effects
+			(font
+				(size 1.27 1.27)
+			)
+			(justify left bottom)
+		)
+	)
+	(text "parts rated\nto 60V !!!"
+		(exclude_from_sim no)
+		(at 92.71 161.29 0)
+		(effects
+			(font
+				(size 1.27 1.27)
+			)
+			(justify left bottom)
+		)
+	)
+	(text "from some kind\nof stepstick\nadapter"
+		(exclude_from_sim no)
+		(at 34.29 93.98 0)
+		(effects
+			(font
+				(size 1.27 1.27)
+			)
+			(justify right bottom)
+		)
+	)
+	(text "\"hybrid\" stepper\nor normal bldc"
+		(exclude_from_sim no)
+		(at 261.62 125.73 0)
+		(effects
+			(font
+				(size 1.27 1.27)
+			)
+			(justify left bottom)
+		)
+	)
 	(junction
 		(at 106.68 177.8)
@@
 		)
 	)
-	(text "this pinout should work\nfor all pre-wired steppers\nAABB\nABAB"
-		(exclude_from_sim no)
-		(at 255.27 121.92 0)
-		(effects
-			(font
-				(size 1.27 1.27)
-			)
-			(justify left bottom)
-		)
-	)
-	(text "parts rated\nto 60V !!!"
-		(exclude_from_sim no)
-		(at 92.71 161.29 0)
-		(effects
-			(font
-				(size 1.27 1.27)
-			)
-			(justify left bottom)
-		)
-	)
-	(text "from some kind\nof stepstick\nadapter"
-		(exclude_from_sim no)
-		(at 34.29 93.98 0)
-		(effects
-			(font
-				(size 1.27 1.27)
-			)
-			(justify right bottom)
-		)
-	)
-	(text "\"hybrid\" stepper\nor normal bldc"
-		(exclude_from_sim no)
-		(at 261.62 125.73 0)
-		(effects
-			(font
-				(size 1.27 1.27)
-			)
-			(justify left bottom)
-		)
-	)
 	(netclass_flag ""
 		(length 2.54)
@@
 		(at 31.75 121.92)
 		(size 30.48 27.94)
+		(exclude_from_sim no)
+		(in_bom yes)
+		(on_board yes)
+		(dnp no)
 		(fields_autoplaced yes)
 		(stroke
@@
 		(at 31.75 36.83)
 		(size 30.48 27.94)
+		(exclude_from_sim no)
+		(in_bom yes)
+		(on_board yes)
+		(dnp no)
 		(fields_autoplaced yes)
 		(stroke
@@
 		(at 193.04 114.3)
 		(size 53.34 34.29)
+		(exclude_from_sim no)
+		(in_bom yes)
+		(on_board yes)
+		(dnp no)
 		(fields_autoplaced yes)
 		(stroke
@@
 		(at 92.71 36.83)
 		(size 43.18 111.76)
+		(exclude_from_sim no)
+		(in_bom yes)
+		(on_board yes)
+		(dnp no)
 		(fields_autoplaced yes)
 		(stroke
@@
 		(at 167.64 36.83)
 		(size 38.1 39.37)
+		(exclude_from_sim no)
+		(in_bom yes)
+		(on_board yes)
+		(dnp no)
 		(fields_autoplaced yes)
 		(stroke
@@
 		(at 158.75 114.3)
 		(size 26.67 34.29)
+		(exclude_from_sim no)
+		(in_bom yes)
+		(on_board yes)
+		(dnp no)
 		(fields_autoplaced yes)
 		(stroke
@@
 		)
 	)
+	(embedded_fonts no)
 )

Commit message: add hybrid board outline
Parts:
- H101: footprint mechanical:NEMA14 -> matei-kicad-footprints:nema-14-17-hybrid
Changed lines of the file:
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@@
 			)
 		)
-		(property "Footprint" "mechanical:NEMA14"
+		(property "Footprint" "matei-kicad-footprints:nema-14-17-hybrid"
 			(at 261.62 64.77 0)
 			(effects
