File: hardware/lemon-pepper.kicad_sch (KiCad schematic)
At the start: 21 parts, among them J101 INPUT, M101 MOT

Commit message: clean erc drc, pack sym, footprints into standalone lib
Parts:
- C101, C102, C103, C104, C105, C106, C107, C108: footprint Capacitor_SMD:C_0805_2012Metric -> lemon-pepper-footprints:C_0805_2012Metric; symbol Device:C_Small -> lemon-pepper-symbols:C_Small
- D101: footprint Diode_SMD:D_SMA -> lemon-pepper-footprints:D_SMA; symbol Device:D -> lemon-pepper-symbols:D
- FID101, FID102, FID103: symbol Mechanical:Fiducial -> lemon-pepper-symbols:Fiducial
- H101: symbol Mechanical:MountingHole_Pad -> lemon-pepper-symbols:MountingHole_Pad
- J101: footprint Connector_JST:JST_XH_B4B-XH-A_1x04_P2.50mm_Vertical -> lemon-pepper-footprints:JST_XH_B4B-XH-A_1x04_P2.50mm_Vertical; symbol Connector_Generic:Conn_01x04 -> lemon-pepper-symbols:Conn_01x04
- JP101: symbol Jumper:SolderJumper_2_Open -> lemon-pepper-symbols:SolderJumper_2_Open
- M101: footprint footprints:XH2.54 4P -> lemon-pepper-footprints:XH2.54 4P; symbol Motor:Stepper_Motor_bipolar -> lemon-pepper-symbols:Stepper_Motor_bipolar
- R101, R102, R103, R104, R105: footprint Resistor_SMD:R_0402_1005Metric -> lemon-pepper-footprints:R_0402_1005Metric; symbol Device:R_Small_US -> lemon-pepper-symbols:R_Small_US
