File: hardware/encoder.kicad_sch (KiCad schematic)
At the start: 3 parts, among them U401 MT6835

Commit message: update to kicad 9
Parts:
- U401: footprint matei:MagnTek TSSOP-16-1EP_4.4x5mm_P0.65mm -> Package_SO:TSSOP-16_4.4x5mm_P0.65mm
Changed lines of the file:
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@@
 (kicad_sch
-	(version 20231120)
+	(version 20250114)
 	(generator "eeschema")
-	(generator_version "8.0")
+	(generator_version "9.0")
 	(paper "A4")
 	(title_block
@@
 		(shape output)
 		(at 119.38 83.82 180)
-		(fields_autoplaced yes)
 		(effects
 			(font
@@
 		(shape output)
 		(at 172.72 96.52 0)
-		(fields_autoplaced yes)
 		(effects
 			(font
@@
 		(shape output)
 		(at 172.72 93.98 0)
-		(fields_autoplaced yes)
 		(effects
 			(font
@@
 		(shape input)
 		(at 119.38 96.52 180)
-		(fields_autoplaced yes)
 		(effects
 			(font
@@
 		(shape input)
 		(at 119.38 88.9 180)
-		(fields_autoplaced yes)
 		(effects
 			(font
@@
 		(shape output)
 		(at 172.72 91.44 0)
-		(fields_autoplaced yes)
 		(effects
 			(font
@@
 		(shape input)
 		(at 119.38 86.36 180)
-		(fields_autoplaced yes)
 		(effects
 			(font
@@
 		(shape input)
 		(at 100.33 91.44 180)
-		(fields_autoplaced yes)
 		(effects
 			(font
@@
 			)
 		)
-		(property "Footprint" "matei:MagnTek TSSOP-16-1EP_4.4x5mm_P0.65mm"
+		(property "Footprint" "Package_SO:TSSOP-16_4.4x5mm_P0.65mm"
 			(at 146.05 96.52 0)
 			(effects

Commit message: clean erc drc, pack sym, footprints into standalone lib
Parts:
- C401: footprint Capacitor_SMD:C_0402_1005Metric -> lemon-pepper-footprints:C_0402_1005Metric; symbol Device:C_Small -> lemon-pepper-symbols:C_Small
- R401: footprint Resistor_SMD:R_0402_1005Metric -> lemon-pepper-footprints:R_0402_1005Metric; symbol Device:R_Small_US -> lemon-pepper-symbols:R_Small_US
- U401: footprint Package_SO:TSSOP-16_4.4x5mm_P0.65mm -> lemon-pepper-footprints:TSSOP-16_4.4x5mm_P0.65mm; symbol matei:MT6835 -> lemon-pepper-symbols:MT6835
Changed lines of the file:
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@@
 			)
 		)
-		(property "Description" ""
+		(property "Description" "Power symbol creates a global label with name \"GND\" , ground"
 			(at 146.05 110.49 0)
 			(effects
@@
 			)
 		)
-		(property "Description" ""
+		(property "Description" "Power symbol creates a global label with name \"GND\" , ground"
 			(at 172.72 83.82 0)
 			(effects
@@
 			)
 		)
-		(property "Description" ""
+		(property "Description" "Power symbol creates a global label with name \"+3V3\""
 			(at 146.05 69.85 0)
 			(effects
@@
 	)
 	(symbol
-		(lib_id "Device:R_Small_US")
+		(lib_id "lemon-pepper-symbols:R_Small_US")
 		(at 107.95 86.36 0)
 		(mirror y)
@@
 			)
 		)
-		(property "Footprint" "Resistor_SMD:R_0402_1005Metric"
+		(property "Footprint" "lemon-pepper-footprints:R_0402_1005Metric"
 			(at 107.95 86.36 0)
 			(effects
@@
 			)
 		)
-		(property "Description" ""
+		(property "Description" "Resistor, small US symbol"
 			(at 107.95 86.36 0)
 			(effects
@@
 	)
 	(symbol
-		(lib_id "Device:C_Small")
+		(lib_id "lemon-pepper-symbols:C_Small")
 		(at 172.72 78.74 0)
 		(unit 1)
@@
 			)
 		)
-		(property "Footprint" "Capacitor_SMD:C_0402_1005Metric"
+		(property "Footprint" "lemon-pepper-footprints:C_0402_1005Metric"
 			(at 172.72 78.74 0)
 			(effects
@@
 			)
 		)
-		(property "Description" ""
+		(property "Description" "Unpolarized capacitor, small symbol"
 			(at 172.72 78.74 0)
 			(effects
@@
 			)
 		)
-		(property "Description" ""
+		(property "Description" "Power symbol creates a global label with name \"+3V3\""
 			(at 107.95 81.28 0)
 			(effects
@@
 	)
 	(symbol
-		(lib_id "matei:MT6835")
+		(lib_id "lemon-pepper-symbols:MT6835")
 		(at 146.05 96.52 0)
 		(unit 1)
@@
 			)
 		)
-		(property "Footprint" "Package_SO:TSSOP-16_4.4x5mm_P0.65mm"
+		(property "Footprint" "lemon-pepper-footprints:TSSOP-16_4.4x5mm_P0.65mm"
 			(at 146.05 96.52 0)
 			(effects
