File: hardware/halfbridges.kicad_sch (KiCad schematic)
At the start: 7 parts, among them U601 L6226QTR

Commit message: clean erc drc, pack sym, footprints into standalone lib
Parts:
- C601, C602: footprint Capacitor_SMD:C_0402_1005Metric -> lemon-pepper-footprints:C_0402_1005Metric; symbol Device:C_Small -> lemon-pepper-symbols:C_Small
- D601: footprint Diode_SMD:D_0603_1608Metric -> lemon-pepper-footprints:D_0603_1608Metric; symbol Device:LED -> lemon-pepper-symbols:LED
- D602, D603: footprint Diode_SMD:D_SOD-323 -> lemon-pepper-footprints:D_SOD-323; symbol Device:D_Small -> lemon-pepper-symbols:D_Small
- R601: footprint Resistor_SMD:R_0402_1005Metric -> lemon-pepper-footprints:R_0402_1005Metric; symbol Device:R_Small_US -> lemon-pepper-symbols:R_Small_US
- U601: footprint matei:ST-L6226Q-VQFN32 -> lemon-pepper-footprints:ST-L6226Q-VQFN32; symbol easyeda2kicad:L6226QTR -> lemon-pepper-symbols:L6226QTR
Connections:
- now unconnected: U601.10 (NC), U601.18 (NC), U601.32 (NC)
Changed lines of the file:
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@@
 	)
 	(symbol
-		(lib_id "easyeda2kicad:L6226QTR")
+		(lib_id "lemon-pepper-symbols:L6226QTR")
 		(at 137.16 91.44 0)
 		(unit 1)
@@
 			)
 		)
-		(property "Footprint" "matei:ST-L6226Q-VQFN32"
+		(property "Footprint" "lemon-pepper-footprints:ST-L6226Q-VQFN32"
 			(at 137.16 129.54 0)
 			(effects
@@
 	)
 	(symbol
-		(lib_id "matei:Vmot")
+		(lib_id "power:+24V")
 		(at 158.75 55.88 0)
 		(unit 1)
@@
 			)
 		)
-		(property "Description" ""
+		(property "Description" "Power symbol creates a global label with name \"+24V\""
 			(at 158.75 55.88 0)
 			(effects
@@
 			)
 		)
-		(property "Description" ""
+		(property "Description" "Power symbol creates a global label with name \"GND\" , ground"
 			(at 158.75 116.84 0)
 			(effects
@@
 	)
 	(symbol
-		(lib_id "Device:R_Small_US")
+		(lib_id "lemon-pepper-symbols:R_Small_US")
 		(at 97.79 99.06 270)
 		(mirror x)
@@
 			)
 		)
-		(property "Footprint" "Resistor_SMD:R_0402_1005Metric"
+		(property "Footprint" "lemon-pepper-footprints:R_0402_1005Metric"
 			(at 97.79 99.06 0)
 			(effects
@@
 			)
 		)
-		(property "Description" ""
+		(property "Description" "Resistor, small US symbol"
 			(at 97.79 99.06 0)
 			(effects
@@
 	)
 	(symbol
-		(lib_id "Device:D_Small")
+		(lib_id "lemon-pepper-symbols:D_Small")
 		(at 139.7 58.42 0)
 		(unit 1)
@@
 			)
 		)
-		(property "Footprint" "Diode_SMD:D_SOD-323"
+		(property "Footprint" "lemon-pepper-footprints:D_SOD-323"
 			(at 139.7 58.42 90)
 			(effects
@@
 			)
 		)
-		(property "Description" ""
+		(property "Description" "Diode, small symbol"
 			(at 139.7 58.42 0)
 			(effects
@@
 	)
 	(symbol
-		(lib_id "Device:C_Small")
+		(lib_id "lemon-pepper-symbols:C_Small")
 		(at 149.86 68.58 90)
 		(mirror x)
@@
 			)
 		)
-		(property "Footprint" "Capacitor_SMD:C_0402_1005Metric"
+		(property "Footprint" "lemon-pepper-footprints:C_0402_1005Metric"
 			(at 149.86 68.58 0)
 			(effects
@@
 			)
 		)
-		(property "Description" ""
+		(property "Description" "Unpolarized capacitor, small symbol"
 			(at 149.86 68.58 0)
 			(effects
@@
 	)
 	(symbol
-		(lib_id "Device:C_Small")
+		(lib_id "lemon-pepper-symbols:C_Small")
 		(at 129.54 63.5 0)
 		(unit 1)
@@
 			)
 		)
-		(property "Footprint" "Capacitor_SMD:C_0402_1005Metric"
+		(property "Footprint" "lemon-pepper-footprints:C_0402_1005Metric"
 			(at 129.54 63.5 0)
 			(effects
@@
 			)
 		)
-		(property "Description" ""
+		(property "Description" "Unpolarized capacitor, small symbol"
 			(at 129.54 63.5 0)
 			(effects
@@
 	)
 	(symbol
-		(lib_id "Device:D_Small")
+		(lib_id "lemon-pepper-symbols:D_Small")
 		(at 139.7 68.58 0)
 		(mirror y)
@@
 			)
 		)
-		(property "Footprint" "Diode_SMD:D_SOD-323"
+		(property "Footprint" "lemon-pepper-footprints:D_SOD-323"
 			(at 139.7 68.58 90)
 			(effects
@@
 			)
 		)
-		(property "Description" ""
+		(property "Description" "Diode, small symbol"
 			(at 139.7 68.58 0)
 			(effects
@@
 			)
 		)
-		(property "Description" ""
+		(property "Description" "Power symbol creates a global label with name \"+3V3\""
 			(at 92.71 96.52 0)
 			(effects
@@
 	)
 	(symbol
-		(lib_id "Device:LED")
+		(lib_id "lemon-pepper-symbols:LED")
 		(at 107.95 99.06 180)
 		(unit 1)
@@
 			)
 		)
-		(property "Footprint" "Diode_SMD:D_0603_1608Metric"
+		(property "Footprint" "lemon-pepper-footprints:D_0603_1608Metric"
 			(at 107.95 99.06 0)
 			(effects
@@
 			)
 		)
-		(property "Description" ""
+		(property "Description" "Light emitting diode"
 			(at 107.95 99.06 0)
 			(effects
@@
 			(at 107.95 99.06 0)
 			(effects
+				(font
+					(size 1.27 1.27)
+				)
+				(hide yes)
+			)
+		)
+		(property "Sim.Pins" "1=K 2=A"
+			(at 107.95 99.06 0)
+			(effects
